File: EL87.sch (KiCad schematic (older format))
At the start: 289 parts, among them U1 proton_c

Commit message: gridified schematic leds might need to be moved on pcb to be more linear
Parts:
- SW1: renamed from SW_1; value MX_LED -> ESC
- SW10: renamed from SW_11; value MX_LED -> F12
- SW11: renamed from SW_14; value MX_LED -> ScrlLck
- SW12: renamed from SW_16; value MX_LED -> PauseBrk
- SW13: renamed from SW_18; value MX_LED -> 1
- SW14: renamed from SW_19; value MX_LED -> F2
- SW15: renamed from SW_20; value MX_LED -> 4
- SW16: renamed from SW_21; value MX_LED -> 5
- SW17: renamed from SW_22; value MX_LED -> 7
- SW18: renamed from SW_25; value MX_LED -> 8
- SW19: renamed from SW_8; value MX_LED -> F8
- SW2: renamed from SW_2; value MX_LED -> F1
- SW20: renamed from SW_28; value MX_LED -> -
- SW21: renamed from SW_29; value MX_LED -> Backspace_2; footprint Keyboard:MXALPS -> Keyboard:MXALPS_2U
- SW22: renamed from SW_12; value MX_LED -> PrntScrn
- SW23: renamed from SW_15; value MX_LED -> /
- SW24: renamed from SW_17; value MX_LED -> extra
- SW25: renamed from SW_36; value MX_LED -> `
- SW26: renamed from SW_37; value MX_LED -> 2
- SW27: renamed from SW_38; value MX_LED -> W
- SW28: renamed from SW_39; value MX_LED -> 6
- SW29: renamed from SW_23; value MX_LED -> Y
- SW3: renamed from SW_3; value MX_LED -> F3
- SW30: renamed from SW_26; value MX_LED -> 9
- SW31: renamed from SW_27; value MX_LED -> F9
- SW32: renamed from SW_46; value MX_LED -> =
- SW33: renamed from SW_30; value MX_LED -> ]
- SW34: renamed from SW_13; value MX_LED -> NumLock
- SW35: renamed from SW_33; value MX_LED -> 8
- SW36: renamed from SW_34; value MX_LED -> *
- SW37: renamed from SW_54; value MX_LED -> Tab_15; footprint Keyboard:MXALPS -> Keyboard:MXALPS_1.5U
- SW38: renamed from SW_55; value MX_LED -> 3
- SW39: renamed from SW_56; value MX_LED -> E
- SW4: renamed from SW_4; value MX_LED -> F4
- SW40: renamed from SW_40; value MX_LED -> R
- SW41: renamed from SW_24; value MX_LED -> U
- SW42: renamed from SW_44; value MX_LED -> I
- SW43: renamed from SW_45; value MX_LED -> 0
- SW44: renamed from SW_47; value MX_LED -> P
- SW45: renamed from SW_48; value MX_LED -> \\_15; footprint Keyboard:MXALPS -> Keyboard:MXALPS_1.5U
- SW46: renamed from SW_31; value MX_LED -> 7
- SW47: renamed from SW_51; value MX_LED -> 5
- SW48: renamed from SW_35; value MX_LED -> -
- SW49: renamed from SW_70; value MX_LED -> Caps_175; footprint Keyboard:MXALPS -> Keyboard:MXALPS_1.75U
- SW5: renamed from SW_5; value MX_LED -> F5
- SW50: renamed from SW_71; value MX_LED -> Q
- SW51: renamed from SW_57; value MX_LED -> S
- SW52: renamed from SW_41; value MX_LED -> T
- SW53: renamed from SW_42; value MX_LED -> H
- SW54: renamed from SW_62; value MX_LED -> J
- SW55: renamed from SW_63; value MX_LED -> O
- SW56: renamed from SW_65; value MX_LED -> [
- SW57: renamed from SW_49; value MX_LED -> '
- SW58: renamed from SW_32; value MX_LED -> 4
- SW59: renamed from SW_52; value MX_LED -> 2
- SW6: renamed from SW_6; value MX_LED -> F6
- SW60: renamed from SW_53; value MX_LED -> 9
- SW61: renamed from SW_86; value MX_LED -> Shift_225; footprint Keyboard:MXALPS -> Keyboard:MXALPS_2.25U
- SW62: renamed from SW_72; value MX_LED -> A
- SW63: renamed from SW_58; value MX_LED -> D
- SW64: renamed from SW_59; value MX_LED -> F
- SW65: renamed from SW_43; value MX_LED -> B
- SW66: renamed from SW_78; value MX_LED -> K
- SW67: renamed from SW_64; value MX_LED -> L
- SW68: renamed from SW_92; value MX_LED -> ;
- SW69: renamed from SW_66; value MX_LED -> Enter_225; footprint Keyboard:MXALPS -> Keyboard:MXALPS_2.25U
- SW7: renamed from SW_7; value MX_LED -> F7
- SW70: renamed from SW_50; value MX_LED -> 1
- SW71: renamed from SW_69; value MX_LED -> 3
- SW72: renamed from SW_85; value MX_LED -> +_2V
- SW73: renamed from SW_87; value MX_LED -> Ctl_125; footprint Keyboard:MXALPS -> Keyboard:MXALPS_1.25U
- SW74: renamed from SW_73; value MX_LED -> Z
- SW75: renamed from SW_74; value MX_LED -> X
- SW76: renamed from SW_60; value MX_LED -> G
- SW77: renamed from SW_61; value MX_LED -> N
- SW78: renamed from SW_79; value MX_LED -> M
- SW79: renamed from SW_80; value MX_LED -> >
- SW8: renamed from SW_9; value MX_LED -> F10
- SW80: renamed from SW_93; value MX_LED -> /
- SW81: renamed from SW_81; value MX_LED -> Shift_275; footprint Keyboard:MXALPS -> Keyboard:MXALPS_2.75U
- SW82: renamed from SW_67; value MX_LED -> 0
- SW83: renamed from SW_84; value MX_LED -> 00
- SW84: renamed from SW_96; value MX_LED -> 6
- SW85: renamed from SW_88; value MX_LED -> OS
- SW86: renamed from SW_89; value MX_LED -> Alt_125; footprint Keyboard:MXALPS -> Keyboard:MXALPS_1.25U
- SW87: renamed from SW_75; value MX_LED -> C
- SW88: renamed from SW_76; value MX_LED -> V
- SW89: renamed from SW_77; value MX_LED -> SPACE_7; footprint Keyboard:MXALPS -> Keyboard:MXALPS_7U
- SW9: renamed from SW_10; value MX_LED -> F11
- SW90: renamed from SW_90; value MX_LED -> <
- SW91: renamed from SW_91; value MX_LED -> Alt_125; footprint Keyboard:MXALPS -> Keyboard:MXALPS_1.25U
- SW92: renamed from SW_94; value MX_LED -> Fn
- SW93: renamed from SW_82; value MX_LED -> Menu
- SW94: renamed from SW_68; value MX_LED -> Ctrl_125; footprint Keyboard:MXALPS -> Keyboard:MXALPS_1.25U
- SW95: renamed from SW_83; value MX_LED -> .
- SW96: renamed from SW_95; value MX_LED -> Enter_2V
- renumbered D11 to D10, D14 to D11, D16 to D12, D18 to D13, D19 to D14, D20 to D15, D21 to D16, D22 to D17, D25 to D18, D8 to D19, D28 to D20, D29 to D21, D12 to D22, D15 to D23, D17 to D24, D36 to D25, D37 to D26, D38 to D27, D39 to D28, D23 to D29, D26 to D30, D27 to D31, D46 to D32, D30 to D33, D13 to D34, D33 to D35, D34 to D36, D54 to D37, D55 to D38, D56 to D39, D24 to D41, D44 to D42, D45 to D43, D47 to D44, D48 to D45, D31 to D46, D51 to D47, D35 to D48, D70 to D49, D71 to D50, D57 to D51, D41 to D52, D42 to D53, D62 to D54, D63 to D55, D65 to D56, D49 to D57, D32 to D58, D52 to D59, D53 to D60, D86 to D61, D72 to D62, D58 to D63, D59 to D64, D43 to D65, D78 to D66, D64 to D67, D92 to D68, D66 to D69, D50 to D70, D69 to D71, D85 to D72, D87 to D73, D73 to D74, D74 to D75, D60 to D76, D61 to D77, D79 to D78, D80 to D79, D9 to D8, D93 to D80, D67 to D82, D84 to D83, D96 to D84, D88 to D85, D89 to D86, D75 to D87, D76 to D88, D77 to D89, D10 to D9, D94 to D92, D82 to D93, D68 to D94, D83 to D95, D95 to D96
Connections:
- net col0: now also U1.B5 (PB5); no longer U1.B10 (PB10)
- net col1: now also U1.B4 (PB4); no longer U1.B11 (PB11)
- net col10: now also U1.A8 (PA8); no longer U1.A4 (PA4/SPEAKER1)
- net col11: now also U1.A15 (PA15); no longer U1.B0 (PB0)
- net col2: now also U1.B3 (PB3); no longer U1.B12 (PB12)
- net col3: now also U1.B2 (PB2); no longer U1.B5 (PB5)
- net col4: now also U1.B1 (PB1); no longer U1.B4 (PB4)
- net col5: now also U1.B0 (PB0); no longer U1.A15 (PA15)
- net col6: now also U1.A4 (PA4/SPEAKER1); no longer U1.A8 (PA8)
- net col7: now also U1.A5 (PA5/SPEAKER2); no longer U1.A7 (PA7)
- net col9: now also U1.A7 (PA7); no longer U1.A5 (PA5/SPEAKER2)
- net row1: no longer D26.1 (K)
- net row2: now also D26.1 (K)
- net row4: now also U1.B9 (PB9); no longer U1.B3 (PB3)
- net row5: now also U1.B10 (PB10); no longer U1.B2 (PB2)
- net row6: now also U1.B11 (PB11); no longer U1.B1 (PB1)
- net row7: now also U1.B12 (PB12); no longer U1.B9 (PB9)
- net SIG_1: now reaches LED1.2 (D_OUT), LED2.4 (D_IN)
- net SIG_2: now reaches LED2.2 (D_OUT), LED3.4 (D_IN)
- net SIG_3: now reaches LED3.2 (D_OUT), LED4.4 (D_IN)
- net SIG_4: now reaches LED4.2 (D_OUT), LED5.4 (D_IN)
- net SIG_5: now reaches LED5.2 (D_OUT), LED6.4 (D_IN)
- net SIG_6: now reaches LED6.2 (D_OUT), LED7.4 (D_IN)
- net SIG_7: now reaches LED7.2 (D_OUT), LED8.4 (D_IN)
- net SIG_8: now reaches LED8.2 (D_OUT), LED9.4 (D_IN)
- net SIG_9: now reaches LED10.4 (D_IN), LED9.2 (D_OUT)
- net SIG_10: now reaches LED10.2 (D_OUT), LED11.4 (D_IN)
- net SIG_11: now reaches LED11.2 (D_OUT), LED12.4 (D_IN)
- net SIG_12: now reaches LED12.2 (D_OUT), LED13.4 (D_IN)
- net SIG_13: now reaches LED13.2 (D_OUT), LED14.4 (D_IN)
- net SIG_14: now reaches LED14.2 (D_OUT), LED15.4 (D_IN)
- net SIG_15: now reaches LED15.2 (D_OUT), LED16.4 (D_IN)
- net SIG_16: now reaches LED16.2 (D_OUT), LED17.4 (D_IN)
- net SIG_17: now reaches LED17.2 (D_OUT), LED18.4 (D_IN)
- net SIG_18: now reaches LED18.2 (D_OUT), LED19.4 (D_IN)
- net SIG_19: now reaches LED19.2 (D_OUT), LED20.4 (D_IN)
- net SIG_20: now reaches LED20.2 (D_OUT), LED21.4 (D_IN)
- net SIG_21: now reaches LED21.2 (D_OUT), LED22.4 (D_IN)
- net SIG_22: now reaches LED22.2 (D_OUT), LED23.4 (D_IN)
- net SIG_23: now reaches LED23.2 (D_OUT), LED24.4 (D_IN)
- net SIG_24: now reaches LED24.2 (D_OUT), LED25.4 (D_IN)
- net SIG_25: now reaches LED25.2 (D_OUT), LED26.4 (D_IN)
- net SIG_26: now reaches LED26.2 (D_OUT), LED27.4 (D_IN)
- net SIG_27: now reaches LED27.2 (D_OUT), LED28.4 (D_IN)
- net SIG_28: now reaches LED28.2 (D_OUT), LED29.4 (D_IN)
- net SIG_29: now reaches LED29.2 (D_OUT), LED30.4 (D_IN)
- net SIG_30: now reaches LED30.2 (D_OUT), LED31.4 (D_IN)
- net SIG_31: now reaches LED31.2 (D_OUT), LED32.4 (D_IN)
- net SIG_32: now reaches LED32.2 (D_OUT), LED33.4 (D_IN)
- net SIG_33: now reaches LED33.2 (D_OUT), LED34.4 (D_IN)
- net SIG_34: now reaches LED34.2 (D_OUT), LED35.4 (D_IN)
- net SIG_35: now reaches LED35.2 (D_OUT), LED36.4 (D_IN)
- net SIG_36: now reaches LED36.2 (D_OUT), LED37.4 (D_IN)
- net SIG_37: now reaches LED37.2 (D_OUT), LED38.4 (D_IN)
- net SIG_38: now reaches LED38.2 (D_OUT), LED39.4 (D_IN)
- net SIG_39: now reaches LED39.2 (D_OUT), LED40.4 (D_IN)
- net SIG_40: now reaches LED40.2 (D_OUT), LED41.4 (D_IN)
- net SIG_41: now reaches LED41.2 (D_OUT), LED42.4 (D_IN)
- net SIG_42: now reaches LED42.2 (D_OUT), LED43.4 (D_IN)
- net SIG_43: now reaches LED43.2 (D_OUT), LED44.4 (D_IN)
- net SIG_44: now reaches LED44.2 (D_OUT), LED45.4 (D_IN)
- net SIG_45: now reaches LED45.2 (D_OUT), LED46.4 (D_IN)
- net SIG_46: now reaches LED46.2 (D_OUT), LED47.4 (D_IN)
- net SIG_47: now reaches LED47.2 (D_OUT), LED48.4 (D_IN)
- net SIG_48: now reaches LED48.2 (D_OUT), LED49.4 (D_IN)
- net SIG_49: now reaches LED49.2 (D_OUT), LED50.4 (D_IN)
- net SIG_50: now reaches LED50.2 (D_OUT), LED51.4 (D_IN)
- net SIG_51: now reaches LED51.2 (D_OUT), LED52.4 (D_IN)
- net SIG_52: now reaches LED52.2 (D_OUT), LED53.4 (D_IN)
- net SIG_53: now reaches LED53.2 (D_OUT), LED54.4 (D_IN)
- net SIG_54: now reaches LED54.2 (D_OUT), LED55.4 (D_IN)
- net SIG_55: now reaches LED55.2 (D_OUT), LED56.4 (D_IN)
- net SIG_56: now reaches LED56.2 (D_OUT), LED57.4 (D_IN)
- net SIG_57: now reaches LED57.2 (D_OUT), LED58.4 (D_IN)
- net SIG_58: now reaches LED58.2 (D_OUT), LED59.4 (D_IN)
- net SIG_59: now reaches LED59.2 (D_OUT), LED60.4 (D_IN)
- net SIG_60: now reaches LED60.2 (D_OUT), LED61.4 (D_IN)
- net SIG_61: now reaches LED61.2 (D_OUT), LED62.4 (D_IN)
- net SIG_62: now reaches LED62.2 (D_OUT), LED63.4 (D_IN)
- net SIG_63: now reaches LED63.2 (D_OUT), LED64.4 (D_IN)
- net SIG_64: now reaches LED64.2 (D_OUT), LED65.4 (D_IN)
- net SIG_65: now reaches LED65.2 (D_OUT), LED66.4 (D_IN)
- net SIG_66: now reaches LED66.2 (D_OUT), LED67.4 (D_IN)
- net SIG_67: now reaches LED67.2 (D_OUT), LED68.4 (D_IN)
- net SIG_68: now reaches LED68.2 (D_OUT), LED69.4 (D_IN)
- net SIG_69: now reaches LED69.2 (D_OUT), LED70.4 (D_IN)
- net SIG_70: now reaches LED70.2 (D_OUT), LED71.4 (D_IN)
- net SIG_71: now reaches LED71.2 (D_OUT), LED72.4 (D_IN)
- net SIG_72: now reaches LED72.2 (D_OUT), LED73.4 (D_IN)
- net SIG_73: now reaches LED73.2 (D_OUT), LED74.4 (D_IN)
- net SIG_74: now reaches LED74.2 (D_OUT), LED75.4 (D_IN)
- net SIG_75: now reaches LED75.2 (D_OUT), LED76.4 (D_IN)
- net SIG_76: now reaches LED76.2 (D_OUT), LED77.4 (D_IN)
- net SIG_77: now reaches LED77.2 (D_OUT), LED78.4 (D_IN)
- net SIG_78: now reaches LED78.2 (D_OUT), LED79.4 (D_IN)
- net SIG_79: now reaches LED79.2 (D_OUT), LED80.4 (D_IN)
- net SIG_80: now reaches LED80.2 (D_OUT), LED81.4 (D_IN)
- net SIG_81: now reaches LED81.2 (D_OUT), LED82.4 (D_IN)
- net SIG_82: now reaches LED82.2 (D_OUT), LED83.4 (D_IN)
- net SIG_83: now reaches LED83.2 (D_OUT), LED84.4 (D_IN)
- net SIG_84: now reaches LED84.2 (D_OUT), LED85.4 (D_IN)
- net SIG_85: now reaches LED85.2 (D_OUT), LED86.4 (D_IN)
- net SIG_86: now reaches LED86.2 (D_OUT), LED87.4 (D_IN)
- net SIG_87: now reaches LED87.2 (D_OUT), LED88.4 (D_IN)
- net SIG_88: now reaches LED88.2 (D_OUT), LED89.4 (D_IN)
- net SIG_89: now reaches LED89.2 (D_OUT), LED90.4 (D_IN)
- net SIG_90: now reaches LED90.2 (D_OUT), LED91.4 (D_IN)
- net SIG_91: now reaches LED91.2 (D_OUT), LED92.4 (D_IN)
- net SIG_92: now reaches LED92.2 (D_OUT), LED93.4 (D_IN)
- net SIG_93: now reaches LED93.2 (D_OUT), LED94.4 (D_IN)
- net SIG_94: now reaches LED94.2 (D_OUT), LED95.4 (D_IN)
- net SIG_95: now reaches LED95.2 (D_OUT), LED96.4 (D_IN)
- net SIG_96: now reaches LED96.2 (D_OUT)
- net A3_5v renamed SIG_0
- no-connect marks 16 -> 15
Other:
- moved on the sheet: D1, D10, D11, D12, D13, D14, D15, D16, D17, D18, D19, D2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
