File: EL87.oilu.kicad_pcb (KiCad board)
At the start: 2 copper layers, 381 x 133.4 mm, 289 parts, among them SW1 ESC, SW10 F12, SW11 ScrlLck, SW12 PauseBrk, SW13 1, SW14 F2, SW15 4, SW16 5, SW17 7, SW18 8, SW19 F8, SW2 F1, SW20 -, SW21 Backspace_2, SW22 PrntScrn, SW23 /, SW24 extra, SW25 GRAVE, SW26 2, SW27 W, SW28 6, SW29 Y, SW3 F3, SW30 9, SW31 F9, SW32 =, SW33 ], SW34 NumLock, SW35 8, SW36 *, SW37 Tab_15, SW38 3, SW39 E, SW4 F4, SW40 R, SW41 U, SW42 I, SW43 0, SW44 P, SW45 \_15, SW46 7, SW47 5, SW48 -, SW49 Caps_175, SW5 F5, SW50 Q, SW51 S, SW52 T, SW53 H, SW54 J, SW55 O, SW56 [, SW57 APOSTROPHE, SW58 4, SW59 2, SW6 F6, SW60 9, SW61 Shift_225, SW62 A, SW63 D, SW64 F, SW65 B, SW66 K, SW67 L, SW68 ;, SW69 Enter_225, SW7 F7, SW70 1, SW71 3, SW72 +_2V, SW73 Ctl_125, SW74 Z, SW75 X, SW76 G, SW77 N, SW78 M, SW79 >, SW8 F10, SW80 /, SW81 Shift_275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

Commit message: rerouted traces
Routing:
- net /GND: track 2110.1 -> 2219.4 mm, vias 0 -> 12
- net /row1: track 601.1 -> 521.3 mm, vias 0 -> 4
- net /5V: track 2026.6 -> 2102.4 mm, vias 1 -> 11
- net /col3: track 233.6 -> 290.5 mm, vias 2 -> 4
- net /col4: track 253.0 -> 285.9 mm
- net /SIG_15: track 44.0 -> 14.2 mm, vias 0 -> 2
- net /row6: track 509.5 -> 538.9 mm, vias 4 -> 5
- net /SIG_84: track 49.1 -> 23.0 mm
- net /SIG_60: track 33.4 -> 59.5 mm
- net /SIG_5: track 49.6 -> 23.8 mm, vias 0 -> 2
- net /col2: track 193.2 -> 216.3 mm, vias 2 -> 1
- net /row7: track 475.9 -> 498.7 mm, vias 0 -> 2
- net /SIG_79: track 35.0 -> 14.2 mm, vias 2 -> 0
- net /SIG_32: track 28.9 -> 48.9 mm, vias 2 -> 0
- net /col11: track 520.6 -> 540.4 mm, vias 0 -> 2
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