File: EL87.kicad_pcb (KiCad board)
At the start: 2 copper layers, 381 x 133.4 mm, 289 parts, among them SW1 ESC, SW10 F12, SW11 ScrlLck, SW12 PauseBrk, SW13 1, SW14 F2, SW15 4, SW16 5, SW17 7, SW18 8, SW19 F8, SW2 F1, SW20 -, SW21 Backspace_2, SW22 PrntScrn, SW23 /, SW24 extra, SW25 GRAVE, SW26 2, SW27 W, SW28 6, SW29 Y, SW3 F3, SW30 9, SW31 F9, SW32 =, SW33 ], SW34 NumLock, SW35 8, SW36 *, SW37 Tab_15, SW38 3, SW39 E, SW4 F4, SW40 R, SW41 U, SW42 I, SW43 0, SW44 P, SW45 \_15, SW46 7, SW47 5, SW48 -, SW49 Caps_175, SW5 F5, SW50 Q, SW51 S, SW52 T, SW53 H, SW54 J, SW55 O, SW56 [, SW57 APOSTROPHE, SW58 4, SW59 2, SW6 F6, SW60 9, SW61 Shift_225, SW62 A, SW63 D, SW64 F, SW65 B, SW66 K, SW67 L, SW68 ;, SW69 Enter_225, SW7 F7, SW70 1, SW71 3, SW72 +_2V, SW73 Ctl_125, SW74 Z, SW75 X, SW76 G, SW77 N, SW78 M, SW79 >, SW8 F10, SW80 /, SW81 Shift_275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

Commit message: changed matrix to have columns follow physical rows to make layout easier to understand
Parts:
- added C1: 100nF, Keebio-Parts:MX-1U-0805, B.Cu at (28.6, 57.1)
- added C10: 100nF, Keebio-Parts:MX-1U-0805, B.Cu at (238.1, 57.1)
- added C11: 100nF, Keebio-Parts:MX-1U-0805, B.Cu at (257.2, 57.1)
- added C12: 100nF, Keebio-Parts:MX-1U-0805, B.Cu at (276.2, 57.1)
- added C13: 100nF, Keebio-Parts:MX-1U-0805, B.Cu at (295.3, 57.1)
- added C14: 100nF, Keebio-Parts:MX-1U-0805, B.Cu at (323.9, 57.1)
- added C15: 100nF, Keebio-Parts:MX-1U-0805, B.Cu at (342.9, 57.1)
- added C16: 100nF, Keebio-Parts:MX-1U-0805, B.Cu at (361.9, 57.1)
- added C17: 100nF, Keebio-Parts:MX-1U-0805, B.Cu at (381.0, 57.1)
- added C18: 100nF, Keebio-Parts:MX-1U-0805, B.Cu at (381.0, 85.7)
- added C19: 100nF, Keebio-Parts:MX-1U-0805, B.Cu at (361.9, 85.7)
- added C2: 100nF, Keebio-Parts:MX-1U-0805, B.Cu at (66.7, 57.1)
- added C20: 100nF, Keebio-Parts:MX-1U-0805, B.Cu at (342.9, 85.7)
- added C21: 100nF, Keebio-Parts:MX-1U-0805, B.Cu at (323.9, 85.7)
- added C22: 100nF, Keebio-Parts:MX-1U-0805, B.Cu at (285.8, 85.7)
- added C23: 100nF, Keebio-Parts:MX-1U-0805, B.Cu at (257.2, 85.7)
- added C24: 100nF, Keebio-Parts:MX-1U-0805, B.Cu at (238.1, 85.7)
- added C25: 100nF, Keebio-Parts:MX-1U-0805, B.Cu at (219.1, 85.7)
- added C26: 100nF, Keebio-Parts:MX-1U-0805, B.Cu at (200.0, 85.7)
- added C27: 100nF, Keebio-Parts:MX-1U-0805, B.Cu at (181.0, 85.7)
- added C28: 100nF, Keebio-Parts:MX-1U-0805, B.Cu at (161.9, 85.7)
- added C29: 100nF, Keebio-Parts:MX-1U-0805, B.Cu at (142.9, 85.7)
- added C3: 100nF, Keebio-Parts:MX-1U-0805, B.Cu at (85.7, 57.1)
- added C30: 100nF, Keebio-Parts:MX-1U-0805, B.Cu at (123.8, 85.7)
- added C31: 100nF, Keebio-Parts:MX-1U-0805, B.Cu at (104.8, 85.7)
- added C32: 100nF, Keebio-Parts:MX-1U-0805, B.Cu at (85.7, 85.7)
- added C33: 100nF, Keebio-Parts:MX-1U-0805, B.Cu at (66.7, 85.7)
- added C34: 100nF, Keebio-Parts:MX-1U-0805, B.Cu at (47.6, 85.7)
- added C35: 100nF, Keebio-Parts:MX-1U-0805, B.Cu at (28.6, 85.7)
- added C36: 100nF, Keebio-Parts:MX-1U-0805, B.Cu at (33.3, 104.8)
- added C37: 100nF, Keebio-Parts:MX-1U-0805, B.Cu at (57.1, 104.8)
- added C38: 100nF, Keebio-Parts:MX-1U-0805, B.Cu at (76.2, 104.8)
- added C39: 100nF, Keebio-Parts:MX-1U-0805, B.Cu at (95.2, 104.8)
- added C4: 100nF, Keebio-Parts:MX-1U-0805, B.Cu at (104.8, 57.1)
- added C40: 100nF, Keebio-Parts:MX-1U-0805, B.Cu at (114.3, 104.8)
- added C41: 100nF, Keebio-Parts:MX-1U-0805, B.Cu at (133.3, 104.8)
- added C42: 100nF, Keebio-Parts:MX-1U-0805, B.Cu at (152.4, 104.8)
- added C43: 100nF, Keebio-Parts:MX-1U-0805, B.Cu at (171.4, 104.8)
- added C44: 100nF, Keebio-Parts:MX-1U-0805, B.Cu at (190.5, 104.8)
- added C45: 100nF, Keebio-Parts:MX-1U-0805, B.Cu at (209.6, 104.8)
- added C46: 100nF, Keebio-Parts:MX-1U-0805, B.Cu at (228.6, 104.8)
- added C47: 100nF, Keebio-Parts:MX-1U-0805, B.Cu at (247.7, 104.8)
- added C48: 100nF, Keebio-Parts:MX-1U-0805, B.Cu at (266.7, 104.8)
- added C49: 100nF, Keebio-Parts:MX-1U-0805, B.Cu at (290.5, 104.8)
- added C5: 100nF, Keebio-Parts:MX-1U-0805, B.Cu at (123.8, 57.1)
- added C50: 100nF, Keebio-Parts:MX-1U-0805, B.Cu at (323.9, 104.8)
- added C51: 100nF, Keebio-Parts:MX-1U-0805, B.Cu at (342.9, 104.8)
- added C52: 100nF, Keebio-Parts:MX-1U-0805, B.Cu at (361.9, 104.8)
- added C53: 100nF, Keebio-Parts:MX-1U-0805, B.Cu at (381.0, 114.3)
- added C54: 100nF, Keebio-Parts:MX-1U-0805, B.Cu at (361.9, 123.8)
- added C55: 100nF, Keebio-Parts:MX-1U-0805, B.Cu at (342.9, 123.8)
- added C56: 100nF, Keebio-Parts:MX-1U-0805, B.Cu at (323.9, 123.8)
- added C57: 100nF, Keebio-Parts:MX-1U-0805, B.Cu at (283.4, 123.8)
- added C58: 100nF, Keebio-Parts:MX-1U-0805, B.Cu at (252.4, 123.8)
- added C59: 100nF, Keebio-Parts:MX-1U-0805, B.Cu at (233.4, 123.8)
- added C6: 100nF, Keebio-Parts:MX-1U-0805, B.Cu at (152.4, 57.1)
- added C60: 100nF, Keebio-Parts:MX-1U-0805, B.Cu at (214.3, 123.8)
- added C61: 100nF, Keebio-Parts:MX-1U-0805, B.Cu at (195.3, 123.8)
- added C62: 100nF, Keebio-Parts:MX-1U-0805, B.Cu at (176.2, 123.8)
- added C63: 100nF, Keebio-Parts:MX-1U-0805, B.Cu at (157.2, 123.8)
- added C64: 100nF, Keebio-Parts:MX-1U-0805, B.Cu at (138.1, 123.8)
- added C65: 100nF, Keebio-Parts:MX-1U-0805, B.Cu at (119.1, 123.8)
- added C66: 100nF, Keebio-Parts:MX-1U-0805, B.Cu at (100.0, 123.8)
- added C67: 100nF, Keebio-Parts:MX-1U-0805, B.Cu at (81.0, 123.8)
- added C68: 100nF, Keebio-Parts:MX-1U-0805, B.Cu at (61.9, 123.8)
- added C69: 100nF, Keebio-Parts:MX-1U-0805, B.Cu at (35.7, 123.8)
- added C7: 100nF, Keebio-Parts:MX-1U-0805, B.Cu at (171.4, 57.1)
- added C70: 100nF, Keebio-Parts:MX-1U-0805, B.Cu at (40.5, 142.9)
- added C71: 100nF, Keebio-Parts:MX-1U-0805, B.Cu at (71.4, 142.9)
- added C72: 100nF, Keebio-Parts:MX-1U-0805, B.Cu at (90.5, 142.9)
- added C73: 100nF, Keebio-Parts:MX-1U-0805, B.Cu at (109.5, 142.9)
- added C74: 100nF, Keebio-Parts:MX-1U-0805, B.Cu at (128.6, 142.9)
- added C75: 100nF, Keebio-Parts:MX-1U-0805, B.Cu at (147.6, 142.9)
- added C76: 100nF, Keebio-Parts:MX-1U-0805, B.Cu at (166.7, 142.9)
- added C77: 100nF, Keebio-Parts:MX-1U-0805, B.Cu at (185.7, 142.9)
- added C78: 100nF, Keebio-Parts:MX-1U-0805, B.Cu at (204.8, 142.9)
- added C79: 100nF, Keebio-Parts:MX-1U-0805, B.Cu at (223.8, 142.9)
- added C8: 100nF, Keebio-Parts:MX-1U-0805, B.Cu at (190.5, 57.1)
- added C80: 100nF, Keebio-Parts:MX-1U-0805, B.Cu at (242.9, 142.9)
- added C81: 100nF, Keebio-Parts:MX-1U-0805, B.Cu at (278.6, 142.9)
- added C82: 100nF, Keebio-Parts:MX-1U-0805, B.Cu at (323.9, 142.9)
- added C83: 100nF, Keebio-Parts:MX-1U-0805, B.Cu at (342.9, 142.9)
- added C84: 100nF, Keebio-Parts:MX-1U-0805, B.Cu at (361.9, 142.9)
- added C85: 100nF, Keebio-Parts:MX-1U-0805, B.Cu at (381.0, 152.4)
- added C86: 100nF, Keebio-Parts:MX-1U-0805, B.Cu at (361.9, 161.9)
- added C87: 100nF, Keebio-Parts:MX-1U-0805, B.Cu at (342.9, 161.9)
- added C88: 100nF, Keebio-Parts:MX-1U-0805, B.Cu at (323.9, 161.9)
- added C89: 100nF, Keebio-Parts:MX-1U-0805, B.Cu at (292.9, 161.9)
- added C9: 100nF, Keebio-Parts:MX-1U-0805, B.Cu at (209.6, 57.1)
- added C90: 100nF, Keebio-Parts:MX-1U-0805, B.Cu at (269.1, 161.9)
- added C91: 100nF, Keebio-Parts:MX-1U-0805, B.Cu at (245.3, 161.9)
- added C92: 100nF, Keebio-Parts:MX-1U-0805, B.Cu at (221.5, 161.9)
- added C93: 100nF, Keebio-Parts:MX-1U-0805, B.Cu at (150.0, 161.9)
- added C94: 100nF, Keebio-Parts:MX-1U-0805, B.Cu at (78.6, 161.9)
- added C95: 100nF, Keebio-Parts:MX-1U-0805, B.Cu at (54.8, 161.9)
- added C96: 100nF, Keebio-Parts:MX-1U-0805, B.Cu at (31.0, 161.9)
- SW10: value F12 -> C
- SW11: value ScrlLck -> Shift_275; footprint Keyboard:MXALPS -> Keyboard:MXALPS_2.75U
- SW12: value PauseBrk -> Space_625; footprint Keyboard:MXALPS -> Keyboard:MXALPS_6.25U
- SW13: value 1 -> F1
- SW14: value F2 -> F9
- SW15: value 4 -> GRAVE
- SW16: value 5 -> 8
- SW17: value 7 -> PgUp
- SW18: value 8 -> Y
- SW19: value F8 -> 7
- SW2: value F1 -> F8
- SW20: value - -> F
- SW21: value Backspace_2 -> ENTER_225; footprint Keyboard:MXALPS_2U -> Keyboard:MXALPS_2.25U
- SW22: value PrntScrn -> V
- SW23: value / -> 1
- SW24: value extra -> Alt_125; footprint Keyboard:MXALPS -> Keyboard:MXALPS_1.25U
- SW25: value GRAVE -> F2
- SW26: value 2 -> F10
- SW27: value W -> 1
- SW28: value 6 -> 9
- SW29: value Y -> -
- SW3: value F3 -> ExtNL
- SW30: value 9 -> U
- SW31: value F9 -> 8
- SW32: value = -> G
- SW33: value ] -> 4
- SW34: value NumLock -> B
- SW35: value 8 -> 2
- SW36: value * -> FN_125; footprint Keyboard:MXALPS -> Keyboard:MXALPS_1.25U
- SW37: value Tab_15 -> F3
- SW38: value 3 -> F11
- SW39: value E -> 2
- SW4: value F4 -> 7
- SW40: value R -> 0
- SW41: value U -> Tab_15; footprint Keyboard:MXALPS -> Keyboard:MXALPS_1.5U
- SW43: value 0 -> 9
- SW44: value P -> H
- SW45: value \_15 -> 5
- SW46: value 7 -> N
- SW47: value 5 -> 3
- SW48: value - -> Menu_125; footprint Keyboard:MXALPS -> Keyboard:MXALPS_1.25U
- SW49: value Caps_175 -> F4; footprint Keyboard:MXALPS_1.75U -> Keyboard:MXALPS
- SW5: value F5 -> Home
- SW50: value Q -> F12
- SW51: value S -> 3
- SW52: value T -> -
- SW53: value H -> Q
- SW54: value J -> O
- SW55: value O -> +
- SW56: value [ -> J
- SW57: value APOSTROPHE -> 6
- SW58: value 4 -> M
- SW59: value 2 -> ENTER_2V
- SW6: value F6 -> T
- SW60: value 9 -> Ctrl_125; footprint Keyboard:MXALPS -> Keyboard:MXALPS_1.25U
- SW61: value Shift_225 -> F5; footprint Keyboard:MXALPS_2.25U -> Keyboard:MXALPS
- SW62: value A -> PrtScr
- SW63: value D -> 4
- SW64: value F -> =
- SW65: value B -> W
- SW66: value K -> P
- SW67: value L -> Caps; footprint Keyboard:MXALPS -> Keyboard:MXALPS_1.75U
- SW68: value ; -> K
- SW69: value Enter_225 -> Shift_225
- SW7: value F7 -> \_15; footprint Keyboard:MXALPS -> Keyboard:MXALPS_1.5U
- SW70: value 1 -> ,
- SW71: value 3 -> Crtl_125; footprint Keyboard:MXALPS -> Keyboard:MXALPS_1.25U
- SW72: value +_2V -> 0
- SW73: value Ctl_125 -> F6
- SW74: value Z -> ScrlLck
- SW75: value X -> 5
- SW76: value G -> BckSpc_2; footprint Keyboard:MXALPS -> Keyboard:MXALPS_2U
- SW77: value N -> E
- SW78: value M -> [
- SW79: value > -> A
- SW8: value F10 -> D
- SW80: value / -> L
- SW81: value Shift_275 -> Z; footprint Keyboard:MXALPS_2.75U -> Keyboard:MXALPS
- SW82: value 0 -> .
- SW83: value 00 -> OS_125; footprint Keyboard:MXALPS -> Keyboard:MXALPS_1.25U
- SW84: value 6 -> 00
- SW85: value OS_125 -> F7
- SW86: value Alt_125 -> PsBrk
- SW87: value C -> 6
- SW88: value V -> Insert
- SW89: value SPACE_625 -> R; footprint Keyboard:MXALPS_6.25U -> Keyboard:MXALPS
- SW9: value F11 -> APOSTROPHE
- SW90: value < -> ]
- SW91: value Alt_125 -> S
- SW92: value Fn_125 -> ;
- SW93: value Menu_125 -> X
- SW94: value Ctrl_125 -> /
- SW95: value . -> Alt_125; footprint Keyboard:MXALPS -> Keyboard:MXALPS_1.25U
- SW96: value Enter_2V -> .
- moved SW71 331.5 mm to (31.0, 161.9)
- moved D71 331.5 mm to (36.5, 157.2)
- moved D86 306.6 mm to (367.5, 52.4)
- moved SW86 302.1 mm to (361.9, 57.1)
- moved SW83 288.1 mm to (54.8, 161.9)
- moved D83 288.1 mm to (60.3, 157.2)
- moved SW74 284.7 mm to (342.9, 57.1)
- moved D74 284.7 mm to (348.5, 52.4)
- moved SW95 283.4 mm to (78.6, 161.9)
- moved D95 283.4 mm to (84.1, 157.2)
- moved SW3 276.2 mm to (381.0, 57.1)
- moved D3 276.2 mm to (386.6, 52.4)
- moved SW62 270.3 mm to (323.9, 57.1)
- moved D62 270.3 mm to (329.4, 52.4)
- moved SW69 243.6 mm to (40.5, 142.9)
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Connections:
- LED1 pad 1: /5V -> Net-(C1-Pad2)
- LED10 pad 1: /5V -> Net-(C10-Pad2)
- LED11 pad 1: /5V -> Net-(C11-Pad2)
- LED12 pad 1: /5V -> Net-(C12-Pad2)
- LED13 pad 1: /5V -> Net-(C13-Pad2)
- LED14 pad 1: /5V -> Net-(C14-Pad2)
- LED15 pad 1: /5V -> Net-(C15-Pad2)
- LED16 pad 1: /5V -> Net-(C16-Pad2)
- LED17 pad 1: /5V -> Net-(C17-Pad2)
- LED18 pad 1: /5V -> Net-(C18-Pad2)
- LED19 pad 1: /5V -> Net-(C19-Pad2)
- LED2 pad 1: /5V -> Net-(C2-Pad2)
- LED20 pad 1: /5V -> Net-(C20-Pad2)
- LED21 pad 1: /5V -> Net-(C21-Pad2)
- LED22 pad 1: /5V -> Net-(C22-Pad2)
- LED23 pad 1: /5V -> Net-(C23-Pad2)
- LED24 pad 1: /5V -> Net-(C24-Pad2)
- LED25 pad 1: /5V -> Net-(C25-Pad2)
- LED26 pad 1: /5V -> Net-(C26-Pad2)
- LED27 pad 1: /5V -> Net-(C27-Pad2)
- LED28 pad 1: /5V -> Net-(C28-Pad2)
- LED29 pad 1: /5V -> Net-(C29-Pad2)
- LED3 pad 1: /5V -> Net-(C3-Pad2)
- LED30 pad 1: /5V -> Net-(C30-Pad2)
- LED31 pad 1: /5V -> Net-(C31-Pad2)
- LED32 pad 1: /5V -> Net-(C32-Pad2)
- LED33 pad 1: /5V -> Net-(C33-Pad2)
- LED34 pad 1: /5V -> Net-(C34-Pad2)
- LED35 pad 1: /5V -> Net-(C35-Pad2)
- LED36 pad 1: /5V -> Net-(C36-Pad2)
- LED37 pad 1: /5V -> Net-(C37-Pad2)
- LED38 pad 1: /5V -> Net-(C38-Pad2)
- LED39 pad 1: /5V -> Net-(C39-Pad2)
- LED4 pad 1: /5V -> Net-(C4-Pad2)
- LED40 pad 1: /5V -> Net-(C40-Pad2)
- LED41 pad 1: /5V -> Net-(C41-Pad2)
- LED42 pad 1: /5V -> Net-(C42-Pad2)
- LED43 pad 1: /5V -> Net-(C43-Pad2)
- LED44 pad 1: /5V -> Net-(C44-Pad2)
- LED45 pad 1: /5V -> Net-(C45-Pad2)
- LED46 pad 1: /5V -> Net-(C46-Pad2)
- LED47 pad 1: /5V -> Net-(C47-Pad2)
- LED48 pad 1: /5V -> Net-(C48-Pad2)
- LED49 pad 1: /5V -> Net-(C49-Pad2)
- LED5 pad 1: /5V -> Net-(C5-Pad2)
- LED50 pad 1: /5V -> Net-(C50-Pad2)
- LED51 pad 1: /5V -> Net-(C51-Pad2)
- LED52 pad 1: /5V -> Net-(C52-Pad2)
- LED53 pad 1: /5V -> Net-(C53-Pad2)
- LED54 pad 1: /5V -> Net-(C54-Pad2)
- LED55 pad 1: /5V -> Net-(C55-Pad2)
- LED56 pad 1: /5V -> Net-(C56-Pad2)
- LED57 pad 1: /5V -> Net-(C57-Pad2)
- LED58 pad 1: /5V -> Net-(C58-Pad2)
- LED59 pad 1: /5V -> Net-(C59-Pad2)
- LED6 pad 1: /5V -> Net-(C6-Pad2)
- LED60 pad 1: /5V -> Net-(C60-Pad2)
- LED61 pad 1: /5V -> Net-(C61-Pad2)
- LED62 pad 1: /5V -> Net-(C62-Pad2)
- LED63 pad 1: /5V -> Net-(C63-Pad2)
- LED64 pad 1: /5V -> Net-(C64-Pad2)
- LED65 pad 1: /5V -> Net-(C65-Pad2)
- LED66 pad 1: /5V -> Net-(C66-Pad2)
- LED67 pad 1: /5V -> Net-(C67-Pad2)
- LED68 pad 1: /5V -> Net-(C68-Pad2)
- LED69 pad 1: /5V -> Net-(C69-Pad2)
- LED7 pad 1: /5V -> Net-(C7-Pad2)
- LED70 pad 1: /5V -> Net-(C70-Pad2)
- LED71 pad 1: /5V -> Net-(C71-Pad2)
- LED72 pad 1: /5V -> Net-(C72-Pad2)
- LED73 pad 1: /5V -> Net-(C73-Pad2)
- LED74 pad 1: /5V -> Net-(C74-Pad2)
- LED75 pad 1: /5V -> Net-(C75-Pad2)
- LED76 pad 1: /5V -> Net-(C76-Pad2)
- LED77 pad 1: /5V -> Net-(C77-Pad2)
- LED78 pad 1: /5V -> Net-(C78-Pad2)
- LED79 pad 1: /5V -> Net-(C79-Pad2)
- LED8 pad 1: /5V -> Net-(C8-Pad2)
- LED80 pad 1: /5V -> Net-(C80-Pad2)
- LED81 pad 1: /5V -> Net-(C81-Pad2)
- LED82 pad 1: /5V -> Net-(C82-Pad2)
- LED83 pad 1: /5V -> Net-(C83-Pad2)
- LED84 pad 1: /5V -> Net-(C84-Pad2)
- LED85 pad 1: /5V -> Net-(C85-Pad2)
- LED86 pad 1: /5V -> Net-(C86-Pad2)
- LED87 pad 1: /5V -> Net-(C87-Pad2)
- LED88 pad 1: /5V -> Net-(C88-Pad2)
- LED89 pad 1: /5V -> Net-(C89-Pad2)
- LED9 pad 1: /5V -> Net-(C9-Pad2)
- LED90 pad 1: /5V -> Net-(C90-Pad2)
- LED91 pad 1: /5V -> Net-(C91-Pad2)
- LED92 pad 1: /5V -> Net-(C92-Pad2)
- LED93 pad 1: /5V -> Net-(C93-Pad2)
- LED94 pad 1: /5V -> Net-(C94-Pad2)
- LED95 pad 1: /5V -> Net-(C95-Pad2)
- LED96 pad 1: /5V -> Net-(C96-Pad2)
- LED96 pad 2: /SIG_96 -> (no net)
- U1 pad 3.3V: Net-(U1-Pad3.3V) -> (no net)
- U1 pad A10: Net-(U1-PadA10) -> (no net)
- U1 pad A13: Net-(U1-PadA13) -> (no net)
- U1 pad A14: Net-(U1-PadA14) -> (no net)
- U1 pad A9: Net-(U1-PadA9) -> (no net)
- U1 pad B13: Net-(U1-PadB13) -> (no net)
- U1 pad B14: Net-(U1-PadB14) -> (no net)
- U1 pad B15: Net-(U1-PadB15) -> (no net)
- U1 pad B6: Net-(U1-PadB6) -> (no net)
- U1 pad B7: Net-(U1-PadB7) -> (no net)
- U1 pad CHRG: Net-(U1-PadCHRG) -> (no net)
- U1 pad D+: Net-(U1-PadD+) -> (no net)
- U1 pad D-: Net-(U1-PadD-) -> (no net)
- U1 pad DFU: Net-(U1-PadDFU) -> (no net)
- U1 pad RST: Net-(U1-PadRST) -> (no net)
Routing:
- net /row0: track 345.2 -> 689.8 mm, vias 1 -> 7
- net /row3: track 499.4 -> 761.7 mm, vias 4 -> 10
- net /row7: track 475.9 -> 716.1 mm, vias 0 -> 11
- net /col2: track 193.2 -> 433.0 mm, vias 2 -> 1
- net /row2: track 505.5 -> 732.0 mm, vias 4 -> 6
- net /row5: track 493.3 -> 718.0 mm, vias 0 -> 5
- net /row6: track 509.5 -> 722.4 mm, vias 4 -> 9
- net /row4: track 528.6 -> 733.4 mm, vias 2 -> 7
- net /col9: track 453.3 -> 259.8 mm, vias 2 -> 0
- net /col4: track 253.0 -> 420.9 mm, vias 3 -> 2
- net /5V: track 2026.6 -> 2191.5 mm, vias 1 -> 0
- net /col1: track 194.6 -> 353.2 mm
- net /col6: track 332.9 -> 459.5 mm, vias 4 -> 1
- net /col7: track 359.2 -> 235.7 mm, vias 3 -> 1
- net /GND: track 2110.1 -> 2222.8 mm, vias 0 -> 9
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
Commit message: Updated the PDFs Rerouted some tracks
Parts:
- SW37: footprint Keyboard:MXALPS_1.5U -> Keyboard:MXALPS
- moved D55 10.3 mm to (385.8, 119.9), turned to 180 degrees
- moved D59 10.3 mm to (385.8, 158.0), turned to 180 degrees
- turned C53 to 90 degrees
- turned C85 to 90 degrees
- turned LED53 to 270 degrees
- turned LED85 to 270 degrees
- turned SW55 to 270 degrees
- turned SW59 to 270 degrees
Routing:
- net /5V: track 2191.5 -> 2172.7 mm
- net /SIG_53: track 54.9 -> 39.3 mm
- net /GND: track 2222.8 -> 2237.6 mm
- net /row4: track 733.4 -> 724.2 mm, vias 7 -> 9
- net /SIG_85: track 37.9 -> 29.7 mm
- net /col0: track 202.7 -> 195.2 mm
- net /SIG_84: track 18.1 -> 11.6 mm
- net /SIG_52: track 18.1 -> 11.6 mm
- net /col6: track 459.5 -> 464.6 mm
- net Net-(C10-Pad2): track 4.26 -> 0.00 mm
- net Net-(C12-Pad2): track 4.26 -> 0.00 mm
- net Net-(C11-Pad2): track 4.26 -> 0.00 mm
- net /row2: track 732.0 -> 735.8 mm
- net /col10: track 485.3 -> 489.1 mm
- net Net-(C85-Pad2): track 2.44 -> 0.00 mm
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
Commit message: Added alternative layouts
Parts:
- removed D23, D83: D, SMD Diodes:D_SOD-123_HandSoldering
- added 6.25U_stab: 6.25U, Keebio-Parts:6.25UReversedStabs, F.Cu at (150.0, 161.9)
- added 7U_STAB: 7U, Keyboard:7U, F.Cu at (161.9, 161.9)
- added C100: 100nF, Keebio-Parts:MX-1U-0805, B.Cu at (32.1, 161.9)
- added C97: 100nF, Keebio-Parts:MX-1U-0805, B.Cu at (150.0, 161.9)
- added C98: 100nF, Keebio-Parts:MX-1U-0805, B.Cu at (79.8, 161.9)
- added C99: 100nF, Keebio-Parts:MX-1U-0805, B.Cu at (56.0, 161.9)
- added C_97: 100nF, Keebio-Parts:MX-1U-0805, B.Cu at (161.9, 161.9)
- added D100: D, SMD Diodes:D_SOD-123_HandSoldering, B.Cu at (25.4, 166.7)
- added D97: D, SMD Diodes:D_SOD-123_HandSoldering, B.Cu at (144.5, 166.7)
- added D98: D, SMD Diodes:D_SOD-123_HandSoldering, B.Cu at (73.0, 166.7)
- added D99: D, SMD Diodes:D_SOD-123_HandSoldering, B.Cu at (49.2, 166.7)
- added ENTER_STAB1: 2.25U, Keebio-Parts:2.25U, F.Cu at (283.4, 123.8)
- added JP1: SOLDER_JUMPER_2, keyboard_parts:SOLDER_JUMPER_2, B.Cu at (227.8, 157.2)
- added JP2: SOLDER_JUMPER_2, keyboard_parts:SOLDER_JUMPER_2, B.Cu at (267.5, 132.6)
- added JP3: SOLDER_JUMPER_2, keyboard_parts:SOLDER_JUMPER_2, B.Cu at (281.4, 134.9)
- added JP4: SOLDER_JUMPER_2, keyboard_parts:SOLDER_JUMPER_2, B.Cu at (287.3, 134.9)
- added JP5: SOLDER_JUMPER_2, keyboard_parts:SOLDER_JUMPER_2, B.Cu at (290.9, 75.4)
- added JP6: SOLDER_JUMPER_2, keyboard_parts:SOLDER_JUMPER_2, B.Cu at (284.2, 75.4)
- added JP7: SOLDER_JUMPER_2, keyboard_parts:SOLDER_JUMPER_2, B.Cu at (267.9, 75.4)
- added LED100: SK6812Mini-E, Keebio-Parts:MX-1U-KS6812Mini-E, F.Cu at (32.1, 161.9)
- added LED97: SK6812Mini-E, Keebio-Parts:MX-1U-KS6812Mini-E, F.Cu at (150.0, 161.9)
- added LED98: SK6812Mini-E, Keebio-Parts:MX-1U-KS6812Mini-E, F.Cu at (79.8, 161.9)
- added LED99: SK6812Mini-E, Keebio-Parts:MX-1U-KS6812Mini-E, F.Cu at (56.0, 161.9)
- added LED_97: SK6812Mini-E, Keebio-Parts:MX-1U-KS6812Mini-E, F.Cu at (161.9, 161.9)
- added NUMPAD_STAB1: 2.25U, Keebio-Parts:2.25U, F.Cu at (381.0, 152.4)
- added NUMPAD_STAB2: 2.25U, Keebio-Parts:2.25U, F.Cu at (381.0, 114.3)
- added STAB99: 2.75U, Keebio-Parts:2.75U, F.Cu at (278.6, 142.9)
- added STAB_2: 2.25U, Keebio-Parts:2.25U, F.Cu at (285.8, 85.7)
- added SW100: CTRL_1.25, Keyboard:MXALPS_1.25U, F.Cu at (31.0, 161.9)
- added SW97: SPACE_6.25, Keyboard:MXALPS, F.Cu at (150.0, 161.9)
- added SW98: ALT_1.25, Keyboard:MXALPS_1.25U, F.Cu at (78.6, 161.9)
- added SW99: GUI_1.25, Keyboard:MXALPS_1.25U, F.Cu at (54.8, 161.9)
- added SW_100: CTRL_1.5, Keyboard:MXALPS_1.5U, F.Cu at (33.3, 161.9)
- added SW_93: CTRL_1.5, Keyboard:MXALPS_1.5U, F.Cu at (290.5, 161.9)
- added SW_94: GUI, Keyboard:MXALPS, F.Cu at (266.7, 161.9)
- added SW_95: ALT_1.5, Keyboard:MXALPS_1.5U, F.Cu at (242.9, 161.9)
- added SW_97: SPACE_7, Keyboard:MXALPS, F.Cu at (161.9, 161.9)
- added SW_98: ALT_1.5, Keyboard:MXALPS_1.5U, F.Cu at (81.0, 161.9)
- added SW_99: GUI, Keyboard:MXALPS, F.Cu at (57.1, 161.9)
- added stab1: 2.25U, Keebio-Parts:2.25U, F.Cu at (40.5, 142.9)
- SW10: value C -> F9
- SW11: value Shift_275 -> F10; footprint Keyboard:MXALPS_2.75U -> Keyboard:MXALPS
- SW12: value Space_625 -> F11; footprint Keyboard:MXALPS_6.25U -> Keyboard:MXALPS
- SW13: value F1 -> F12
- SW14: value F9 -> PrtScrn
- SW15: value GRAVE -> ScrlLck
- SW16: value 8 -> PB
- SW17: value PgUp -> NumLck
- SW18: value Y -> -
- SW19: value 7 -> PgUp; footprint Keyboard:MXALPS -> Keyboard:MXALPS_2.25U
- SW2: value F8 -> F1
- SW20: value F -> Home
- SW21: value ENTER_225 -> Insert; footprint Keyboard:MXALPS_2.25U -> Keyboard:MXALPS
- SW22: value V -> BckSpc_split
- SW24: value Alt_125 -> BckSpc_Split_2; footprint Keyboard:MXALPS_1.25U -> Keyboard:MXALPS
- SW25: value F2 -> =
- SW26: value F10 -> -
- SW27: value 1 -> 0
- SW29: value - -> 8
- SW3: value ExtNL -> F2
- SW30: value U -> 7
- SW31: value 8 -> 6
- SW32: value G -> 5
- SW34: value B -> 3
- SW35: footprint Keyboard:MXALPS -> Keyboard:MXALPS_1.5U
- SW36: value FN_125 -> 1; footprint Keyboard:MXALPS_1.25U -> Keyboard:MXALPS
- SW37: value F3 -> GRAVE
- SW38: value F11 -> Tab_1.5; footprint Keyboard:MXALPS -> Keyboard:MXALPS_1.5U
- SW39: value 2 -> Q
- SW4: value 7 -> F3
- SW40: value 0 -> W
- SW41: value Tab_15 -> E; footprint Keyboard:MXALPS_1.5U -> Keyboard:MXALPS
- SW42: value I -> R
- SW43: value 9 -> T
- SW44: value H -> Y
- SW45: value 5 -> U; footprint Keyboard:MXALPS_1.5U -> Keyboard:MXALPS
- SW46: value N -> I
- SW47: value 3 -> O
- SW48: value Menu_125 -> P; footprint Keyboard:MXALPS_1.25U -> Keyboard:MXALPS
- SW49: value F4 -> [
- SW5: value Home -> F4
- SW50: value F12 -> ]
- SW51: value 3 -> \; footprint Keyboard:MXALPS -> Keyboard:MXALPS_1.5U
- SW52: value - -> DEL
- SW53: value Q -> END
- SW54: value O -> PGDN
- SW56: value J -> 6
- SW57: value 6 -> 5
- SW58: value M -> 4
- SW59: value ENTER_2V -> Enter_2.25
- SW6: value T -> F5
- SW60: value Ctrl_125 -> APOSTROPHE; footprint Keyboard:MXALPS_1.25U -> Keyboard:MXALPS
- SW61: value F5 -> ;
- SW62: value PrtScr -> L
- SW63: value 4 -> K
- SW64: value = -> J; footprint Keyboard:MXALPS -> Keyboard:MXALPS_2U
- SW65: value W -> H
- SW66: value P -> G
- SW67: value Caps -> F; footprint Keyboard:MXALPS_1.75U -> Keyboard:MXALPS
- SW68: value K -> D
- SW69: value Shift_225 -> S; footprint Keyboard:MXALPS_2.25U -> Keyboard:MXALPS
- SW7: value \_15 -> F6
- SW70: value , -> A
- SW71: value Crtl_125 -> CAPS_1.75; footprint Keyboard:MXALPS_1.25U -> Keyboard:MXALPS_1.75U
- SW72: value 0 -> SHIFT_2.25
- SW73: value F6 -> Z; footprint Keyboard:MXALPS_1.25U -> Keyboard:MXALPS
- SW74: value ScrlLck -> X
- SW75: value 5 -> C
- SW76: value BckSpc_2 -> V; footprint Keyboard:MXALPS_2U -> Keyboard:MXALPS
- SW77: value E -> B
- SW78: value [ -> N
- SW79: value A -> M
- SW8: value D -> F7
- SW80: value L -> ,
- SW81: value Z -> .
- SW82: value . -> /
- SW83: value OS_125 -> Shift_split_1.75; footprint Keyboard:MXALPS_1.25U -> Keyboard:MXALPS_1.75U
- SW84: value 00 -> Shift_2.75; footprint Keyboard:MXALPS -> Keyboard:MXALPS_2.75U
- SW85: value F7 -> Shift_split_fn; footprint Keyboard:MXALPS_1.25U -> Keyboard:MXALPS
- SW86: value PsBrk -> 1; footprint Keyboard:MXALPS_1.25U -> Keyboard:MXALPS
- SW87: value 6 -> 2
- SW88: value Insert -> 3
- SW89: value R -> Enter
- SW9: value APOSTROPHE -> F8
- SW90: value ] -> .
- SW91: value S -> 00; footprint Keyboard:MXALPS_1.25U -> Keyboard:MXALPS
- SW92: value ; -> 0; footprint Keyboard:MXALPS_1.25U -> Keyboard:MXALPS
- SW93: value X -> Ctrl_1.25
- SW94: value / -> MENU_1.25
- SW95: value Alt_125 -> GUI_1.25
- SW96: value . -> ALT_1.25; footprint Keyboard:MXALPS -> Keyboard:MXALPS_1.25U
- SW_22: renamed from SW23; value 1 -> BckSpc_2
- moved SW15 315.6 mm to (342.9, 57.1), turned to 180 degrees
- moved D3 306.5 mm to (80.2, 61.9), turned to 90 degrees
- moved D15 303.8 mm to (337.3, 61.9), turned to 90 degrees
- moved SW3 295.3 mm to (85.7, 57.1), turned to 180 degrees
- moved D72 294.6 mm to (34.9, 147.6), turned to 90 degrees
- moved D35 291.3 mm to (61.1, 90.5), turned to 90 degrees
- moved SW53 285.8 mm to (342.9, 104.8), turned to 180 degrees
- moved SW72 284.0 mm to (40.5, 142.9), turned to 180 degrees
- moved SW35 282.1 mm to (66.7, 85.7), turned to 180 degrees
- moved D74 280.2 mm to (84.9, 147.6), turned to 90 degrees
- moved D53 274.8 mm to (337.3, 109.5), turned to 90 degrees
- moved SW89 270.9 mm to (381.0, 152.4), turned to 90 degrees
- moved SW74 266.6 mm to (90.5, 142.9), turned to 180 degrees
- moved SW91 264.7 mm to (342.9, 161.9), turned to 180 degrees
- moved D38 260.3 mm to (27.8, 109.5), turned to 90 degrees
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Connections:
- D11 pad 1: /row0 -> /row1
- D12 pad 1: /row0 -> /row1
- D21 pad 1: /row1 -> /row2
- D22 pad 1: /row1 -> /row2
- D24 pad 1: /row1 -> /row2
- D32 pad 1: /row2 -> /row3
- D33 pad 1: /row2 -> /row3
- D34 pad 1: /row2 -> /row3
- D35 pad 1: /row2 -> /row3
- D36 pad 1: /row2 -> /row3
- D42 pad 1: /row3 -> /row4
- D43 pad 1: /row3 -> /row4
- D44 pad 1: /row3 -> /row4
- D45 pad 1: /row3 -> /row4
- D46 pad 1: /row3 -> /row4
- D47 pad 1: /row3 -> /row4
- D48 pad 1: /row3 -> /row4
- D52 pad 1: /row4 -> /row5
- D53 pad 1: /row4 -> /row5
- D54 pad 1: /row4 -> /row5
- D55 pad 1: /row4 -> /row5
- D56 pad 1: /row4 -> /row5
- D57 pad 1: /row4 -> /row5
- D58 pad 1: /row4 -> /row5
- D59 pad 1: /row4 -> /row5
- D60 pad 1: /row4 -> /row5
- D62 pad 1: /row5 -> /row6
- D63 pad 1: /row5 -> /row6
- D64 pad 1: /row5 -> /row6
- D65 pad 1: /row5 -> /row6
- D66 pad 1: /row5 -> /row6
- D67 pad 1: /row5 -> /row6
- D68 pad 1: /row5 -> /row6
- D69 pad 1: /row5 -> /row6
- D70 pad 1: /row5 -> /row6
- D71 pad 1: /row5 -> /row6
- D72 pad 1: /row5 -> /row7
- D73 pad 1: /row6 -> /row7
- D74 pad 1: /row6 -> /row7
- D75 pad 1: /row6 -> /row7
- D76 pad 1: /row6 -> /row7
- D77 pad 1: /row6 -> /row7
- D78 pad 1: /row6 -> /row7
- D79 pad 1: /row6 -> /row7
- D80 pad 1: /row6 -> /row7
- D81 pad 1: /row6 -> /row7
- D82 pad 1: /row6 -> /row8
- D84 pad 1: /row6 -> /row8
- D85 pad 1: /row7 -> /row8
- D86 pad 1: /row7 -> /row8
- D87 pad 1: /row7 -> /row8
- D88 pad 1: /row7 -> /row8
- D89 pad 1: /row7 -> /row8
- D90 pad 1: /row7 -> /row8
- D91 pad 1: /row7 -> /row8
- D92 pad 1: /row7 -> /row8
- D93 pad 1: /row7 -> /row9
- D94 pad 1: /row7 -> /row9
- D95 pad 1: /row7 -> /row9
- D96 pad 1: /row7 -> /row9
- LED96 pad 2: (no net) -> /SIG_96
- SW11 pad SW1: /col10 -> /col0
- SW12 pad SW1: /col11 -> /col1
- SW13 pad SW1: /col0 -> /col2
- SW14 pad SW1: /col1 -> /col3
- SW15 pad SW1: /col2 -> /col4
- SW16 pad SW1: /col3 -> /col5
- SW17 pad SW1: /col4 -> /col6
- SW18 pad SW1: /col5 -> /col7
- SW19 pad SW1: /col6 -> /col8
- SW20 pad SW1: /col7 -> /col9
- SW21 pad SW1: /col8 -> /col0
- SW22 pad SW1: /col9 -> /col1
- SW24 pad SW1: /col11 -> /col2
- SW25 pad SW1: /col0 -> /col3
- SW26 pad SW1: /col1 -> /col4
- SW27 pad SW1: /col2 -> /col5
- SW28 pad SW1: /col3 -> /col6
- SW29 pad SW1: /col4 -> /col7
- SW30 pad SW1: /col5 -> /col8
- SW31 pad SW1: /col6 -> /col9
- SW32 pad SW1: /col7 -> /col0
- SW33 pad SW1: /col8 -> /col1
- SW34 pad SW1: /col9 -> /col2
- SW35 pad SW1: /col10 -> /col3
- SW36 pad SW1: /col11 -> /col4
- SW37 pad SW1: /col0 -> /col5
- SW38 pad SW1: /col1 -> /col6
- SW39 pad SW1: /col2 -> /col7
- SW40 pad SW1: /col3 -> /col8
- SW41 pad SW1: /col4 -> /col9
- SW42 pad SW1: /col5 -> /col0
- SW43 pad SW1: /col6 -> /col1
- SW44 pad SW1: /col7 -> /col2
- SW45 pad SW1: /col8 -> /col3
- SW46 pad SW1: /col9 -> /col4
- SW47 pad SW1: /col10 -> /col5
- SW48 pad SW1: /col11 -> /col6
- SW49 pad SW1: /col0 -> /col7
- SW50 pad SW1: /col1 -> /col8
- SW51 pad SW1: /col2 -> /col9
- SW52 pad SW1: /col3 -> /col0
- SW53 pad SW1: /col4 -> /col1
- SW54 pad SW1: /col5 -> /col2
- SW55 pad SW1: /col6 -> /col3
- SW56 pad SW1: /col7 -> /col4
- SW57 pad SW1: /col8 -> /col5
- SW58 pad SW1: /col9 -> /col6
- SW59 pad SW1: /col10 -> /col7
- SW60 pad SW1: /col11 -> /col8
- SW61 pad SW1: /col0 -> /col9
- SW62 pad SW1: /col1 -> /col0
- SW63 pad SW1: /col2 -> /col1
- SW64 pad SW1: /col3 -> /col2
- SW65 pad SW1: /col4 -> /col3
- SW66 pad SW1: /col5 -> /col4
- SW67 pad SW1: /col6 -> /col5
- SW68 pad SW1: /col7 -> /col6
- SW69 pad SW1: /col8 -> /col7
- SW70 pad SW1: /col9 -> /col8
- SW71 pad SW1: /col10 -> /col9
- SW72 pad SW1: /col11 -> /col0
- SW73 pad SW1: /col0 -> /col1
- SW74 pad SW1: /col1 -> /col2
- SW75 pad SW1: /col2 -> /col3
- SW76 pad SW1: /col3 -> /col4
- SW77 pad SW1: /col4 -> /col5
- SW78 pad SW1: /col5 -> /col6
- SW79 pad SW1: /col6 -> /col7
- SW80 pad SW1: /col7 -> /col8
- SW81 pad SW1: /col8 -> /col9
- SW82 pad SW1: /col9 -> /col0
- SW83 pad SW1: /col10 -> /col1
- SW83 pad SW2: Net-(D83-Pad2) -> Net-(D84-Pad2)
- SW84 pad SW1: /col11 -> /col1
- SW85 pad SW1: /col0 -> /col2
- SW86 pad SW1: /col1 -> /col3
- SW87 pad SW1: /col2 -> /col4
- SW88 pad SW1: /col3 -> /col5
- SW89 pad SW1: /col4 -> /col6
- SW90 pad SW1: /col5 -> /col7
- SW91 pad SW1: /col6 -> /col8
- SW92 pad SW1: /col7 -> /col9
- SW93 pad SW1: /col8 -> /col0
- SW94 pad SW1: /col9 -> /col1
- SW95 pad SW1: /col10 -> /col2
- SW96 pad SW1: /col11 -> /col3
- SW_22 pad SW1: /col10 -> /col1
- SW_22 pad SW2: Net-(D23-Pad2) -> Net-(D22-Pad2)
- U1 pad 3.3V: (no net) -> Net-(U1-Pad3.3V)
- U1 pad A10: (no net) -> Net-(U1-PadA10)
- U1 pad A13: (no net) -> Net-(U1-PadA13)
- U1 pad A14: (no net) -> Net-(U1-PadA14)
- U1 pad A15: /col11 -> /row8
- U1 pad A8: /col10 -> /row9
- U1 pad A9: (no net) -> Net-(U1-PadA9)
- U1 pad B13: (no net) -> Net-(U1-PadB13)
- U1 pad B14: (no net) -> Net-(U1-PadB14)
- U1 pad B15: (no net) -> Net-(U1-PadB15)
- U1 pad B6: (no net) -> Net-(U1-PadB6)
- U1 pad B7: (no net) -> Net-(U1-PadB7)
- U1 pad CHRG: (no net) -> Net-(U1-PadCHRG)
- U1 pad D+: (no net) -> Net-(U1-PadD+)
- U1 pad D-: (no net) -> Net-(U1-PadD-)
- U1 pad DFU: (no net) -> Net-(U1-PadDFU)
- U1 pad RST: (no net) -> Net-(U1-PadRST)
Routing:
- net /col7: track 235.7 -> 771.8 mm, vias 1 -> 6
- net /row3: track 761.1 -> 247.3 mm, vias 10 -> 1
- net /col5: track 251.5 -> 742.9 mm, vias 1 -> 4
- net /col10: track 489.1 -> 0.00 mm, vias 2 -> 0
- net /row6: track 722.3 -> 236.1 mm, vias 9 -> 5
- net /row0: track 691.0 -> 216.9 mm, vias 7 -> 0
- net /row4: track 724.2 -> 267.8 mm, vias 9 -> 1
- net /row7: track 716.1 -> 278.1 mm, vias 11 -> 3
- net /col0: track 195.2 -> 633.0 mm, vias 0 -> 4
- net /row8: track 0.00 -> 426.9 mm, vias 0 -> 3
- net /row2: track 735.8 -> 315.1 mm, vias 6 -> 0
- net /col11: track 414.1 -> 0.00 mm, vias 1 -> 0
- net /col3: track 316.1 -> 707.6 mm, vias 0 -> 7
- net /row9: track 0.00 -> 361.3 mm, vias 0 -> 1
- net /col6: track 464.6 -> 814.0 mm, vias 1 -> 4
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Other:
- outline, holes or cut-outs redrawn

Commit message: added mounting holes. changed diodes to proper footprint.
Parts:
- added HOLE_M3_1: 1, keyboard_parts:HOLE_M3, F.Cu at (19.1, 171.4)
- added HOLE_M3_2: 2, keyboard_parts:HOLE_M3, F.Cu at (19.1, 47.6)
- added HOLE_M3_3: 3, keyboard_parts:HOLE_M3, F.Cu at (181.0, 57.1)
- added HOLE_M3_4: 4, keyboard_parts:HOLE_M3, F.Cu at (390.5, 47.6)
- added HOLE_M3_5: 5, keyboard_parts:HOLE_M3, F.Cu at (390.5, 171.4)
- added HOLE_M3_6: 6, keyboard_parts:HOLE_M3, F.Cu at (188.1, 161.9)
- D1, D10, D100, D11, D12, D13, D14, D15, D16, D17, D18, D19, D2, D20, D21, D22, D24, D25, D26, D27, D28, D29, D3, D30, D31, D32, D33, D34, D35, D36, D37, D38, D39, D4, D40, D41, D42, D43, D44, D45, D46, D47, D48, D49, D5, D50, D51, D52, D53, D54, D55, D56, D57, D58, D59, D6, D60, D61, D62, D63, D64, D65, D66, D67, D68, D69, D7, D70, D71, D72, D73, D74, D75, D76, D77, D78, D79, D8, D80, D81, D82, D84, D85, D86, D87, D88, D89, D9, D90, D91, D92, D93, D94, D95, D96, D97, D98, D99: footprint SMD Diodes:D_SOD-123_HandSoldering -> Diode_SMD:D_SOD-323_HandSoldering
- STAB_2: value 2.25U -> 2U_stab; footprint Keebio-Parts:2.25U -> Keebio-Parts:2U_stab
Routing:
- net /col7: track 771.8 -> 708.2 mm, vias 6 -> 5
- net /GND: track 2156.4 -> 2212.1 mm, vias 0 -> 2
- net /col8: track 688.4 -> 635.5 mm, vias 6 -> 5
- net /SIG_80: track 31.9 -> 74.0 mm
- net /row1: track 448.4 -> 412.8 mm, vias 0 -> 1
- net /SIG_39: track 64.3 -> 30.4 mm, vias 0 -> 2
- net /col3: track 707.6 -> 738.2 mm, vias 7 -> 5
- net /5V: track 2200.5 -> 2172.7 mm, vias 0 -> 1
- net /SIG_32: track 14.2 -> 41.5 mm
- net /col2: track 660.7 -> 633.7 mm, vias 7 -> 8
- net /row0: track 216.9 -> 243.0 mm
- net /col4: track 643.0 -> 668.8 mm, vias 7 -> 6
- net /col6: track 814.0 -> 788.5 mm
- net /row4: track 267.8 -> 287.7 mm
- net /SIG_36: track 34.1 -> 14.2 mm
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
Commit message: verified LED layout
Parts:
- added HOLE_M3_6: 6, keyboard_parts:HOLE_M3, F.Cu at (181.0, 114.3)
- U1: moved to F.Cu
- moved D55 10.0 mm to (375.4, 119.1)
- moved D89 10.0 mm to (375.4, 157.2)
- turned C55 to 0 degrees
- turned C89 to 0 degrees
- turned HOLE_M3_3 to 0 degrees
- turned LED55 to 180 degrees
- turned LED89 to 180 degrees
- turned SW55 to 180 degrees
- turned SW89 to 180 degrees
- turned U1 to 0 degrees
- renumbered SW_22 to SW23
Routing:
- net /row4: track 287.7 -> 339.1 mm
- net /GND: track 2212.1 -> 2162.2 mm, vias 2 -> 0
- net /SIG_80: track 74.0 -> 31.9 mm
- net /SIG_81: track 30.8 -> 70.9 mm, vias 2 -> 0
- net /col5: track 756.9 -> 718.8 mm, vias 4 -> 7
- net /SIG_87: track 41.7 -> 73.0 mm
- net /col4: track 668.8 -> 640.3 mm, vias 6 -> 5
- net /SIG_32: track 41.5 -> 14.2 mm
- net /row3: track 242.7 -> 269.9 mm, vias 1 -> 0
- net /col0: track 623.6 -> 602.6 mm, vias 6 -> 4
- net /SIG_64: track 20.1 -> 40.7 mm
- net /SIG_30: track 14.2 -> 33.6 mm
- net /SIG_33: track 33.6 -> 14.2 mm
- net /SIG_27: track 33.5 -> 14.2 mm
- net /SIG_35: track 32.6 -> 14.2 mm
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